File: V1/esp-poe-2rl-V1-lan.kicad_sch (KiCad schematic)
At the start: 28 parts, among them J7 ETHERNET, U5 LAN8710A

Commit message: Dev
Other:
- title: ESP 16x 24VDC Input 16x 24VDC Output Module -> ESP 2x Relay Output Module with PoE
Changed lines of the file:
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@@
   (paper "A4")
   (title_block
-    (title "ESP 16x 24VDC Input 16x 24VDC Output Module")
-    (date "2023-05-05")
-    (rev "V2")
+    (title "ESP 2x Relay Output Module with PoE")
+    (date "2023-08-02")
+    (rev "V1")
   )
   (junction (at 266.7 125.73) (diameter 0) (color 0 0 0 0)

Commit message: Working on PoE frontend.
Parts:
- C14: value 1nF/2kV/1206 -> 1nF/2kV
- C15, C18, C19, C20: value 0,1uF/50V/0402 -> 0,1uF/50V
- C16, C17: value 10uF/10V/0603 -> 10uF/10V
- C21: value 1uF/25V/0402 -> 1uF/25V
- C22: value 470pF/50V/0402 -> 470pF/50V
- R15, R18, R19, R20, R21, R22, R23, R25: value 2k2/62,5mW/0402 -> 2k2/62,5mW
- R16, R17: value 330R/62,5mW/0402 -> 330R/62,5mW
- R24: value 10k/62,5mW/0402 -> 10k/62,5mW
- R26: value 12,1k/62,5mW/0402 -> 12,1k/62,5mW
- R27, R28, R29, R30: value 49,9R/62,5mW/0402 -> 49,9R/62,5mW
Changed lines of the file:
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@@
       (effects (font (size 1.27 1.27)) (justify left))
     )
-    (property "Value" "0,1uF/50V/0402" (at 209.55 43.18 0)
+    (property "Value" "0,1uF/50V" (at 209.55 43.18 0)
       (effects (font (size 1.27 1.27)) (justify left))
     )
@@
       (effects (font (size 1.27 1.27)) (justify left))
     )
-    (property "Value" "10k/62,5mW/0402" (at 133.35 121.92 0)
+    (property "Value" "10k/62,5mW" (at 133.35 121.92 0)
       (effects (font (size 1.27 1.27)) (justify left))
     )
@@
       (effects (font (size 1.27 1.27)) (justify left))
     )
-    (property "Value" "330R/62,5mW/0402" (at 53.34 129.54 0)
+    (property "Value" "330R/62,5mW" (at 53.34 129.54 0)
       (effects (font (size 1.27 1.27)) (justify left))
     )
@@
       (effects (font (size 1.27 1.27)) (justify left))
     )
-    (property "Value" "10uF/10V/0603" (at 130.81 32.385 0)
+    (property "Value" "10uF/10V" (at 130.81 32.385 0)
       (effects (font (size 1.27 1.27)) (justify left))
     )
@@
       (effects (font (size 1.27 1.27)) (justify left))
     )
-    (property "Value" "0,1uF/50V/0402" (at 76.2 167.6462 0)
+    (property "Value" "0,1uF/50V" (at 76.2 167.6462 0)
       (effects (font (size 1.27 1.27)) (justify left))
     )
@@
       (effects (font (size 1.27 1.27)) (justify left))
     )
-    (property "Value" "2k2/62,5mW/0402" (at 64.77 53.34 0)
+    (property "Value" "2k2/62,5mW" (at 64.77 53.34 0)
       (effects (font (size 1.27 1.27)) (justify left))
     )
@@
       (effects (font (size 1.27 1.27)) (justify left))
     )
-    (property "Value" "2k2/62,5mW/0402" (at 138.43 53.34 0)
+    (property "Value" "2k2/62,5mW" (at 138.43 53.34 0)
       (effects (font (size 1.27 1.27)) (justify left))
     )
@@
       (effects (font (size 1.27 1.27)) (justify left))
     )
-    (property "Value" "2k2/62,5mW/0402" (at 88.9 53.34 0)
+    (property "Value" "2k2/62,5mW" (at 88.9 53.34 0)
       (effects (font (size 1.27 1.27)) (justify left))
     )
@@
       (effects (font (size 1.27 1.27)) (justify left))
     )
-    (property "Value" "1nF/2kV/1206" (at 50.8 179.0762 0)
+    (property "Value" "1nF/2kV" (at 50.8 179.0762 0)
       (effects (font (size 1.27 1.27)) (justify left))
     )
@@
       (effects (font (size 1.27 1.27)) (justify right))
     )
-    (property "Value" "330R/62,5mW/0402" (at 40.64 129.54 0)
+    (property "Value" "330R/62,5mW" (at 40.64 129.54 0)
       (effects (font (size 1.27 1.27)) (justify right))
     )
@@
       (effects (font (size 1.27 1.27)))
     )
-    (property "Value" "49,9R/62,5mW/0402" (at 252.73 133.35 90)
+    (property "Value" "49,9R/62,5mW" (at 252.73 133.35 90)
       (effects (font (size 1.27 1.27)))
     )
@@
       (effects (font (size 1.27 1.27)) (justify left))
     )
-    (property "Value" "1uF/25V/0402" (at 231.14 43.1862 0)
+    (property "Value" "1uF/25V" (at 231.14 43.1862 0)
       (effects (font (size 1.27 1.27)) (justify left))
     )
@@
       (effects (font (size 1.27 1.27)) (justify left))
     )
-    (property "Value" "2k2/62,5mW/0402" (at 124.46 96.52 0)
+    (property "Value" "2k2/62,5mW" (at 124.46 96.52 0)
       (effects (font (size 1.27 1.27)) (justify left))
     )
@@
       (effects (font (size 1.27 1.27)) (justify left))
     )
-    (property "Value" "0,1uF/50V/0402" (at 153.67 31.75 0)
+    (property "Value" "0,1uF/50V" (at 153.67 31.75 0)
       (effects (font (size 1.27 1.27)) (justify left))
     )
@@
       (effects (font (size 1.27 1.27)))
     )
-    (property "Value" "49,9R/62,5mW/0402" (at 252.73 120.65 90)
+    (property "Value" "49,9R/62,5mW" (at 252.73 120.65 90)
       (effects (font (size 1.27 1.27)))
     )
@@
       (effects (font (size 1.27 1.27)) (justify left))
     )
-    (property "Value" "10uF/10V/0603" (at 133.35 131.445 0)
+    (property "Value" "10uF/10V" (at 133.35 131.445 0)
       (effects (font (size 1.27 1.27)) (justify left))
     )
@@
       (effects (font (size 1.27 1.27)) (justify left))
     )
-    (property "Value" "2k2/62,5mW/0402" (at 107.95 116.84 0)
+    (property "Value" "2k2/62,5mW" (at 107.95 116.84 0)
       (effects (font (size 1.27 1.27)) (justify left))
     )
@@
       (effects (font (size 1.27 1.27)) (justify left))
     )
-    (property "Value" "470pF/50V/0402" (at 251.46 43.18 0)
+    (property "Value" "470pF/50V" (at 251.46 43.18 0)
       (effects (font (size 1.27 1.27)) (justify left))
     )
@@
       (effects (font (size 1.27 1.27)) (justify left))
     )
-    (property "Value" "2k2/62,5mW/0402" (at 97.79 130.81 0)
+    (property "Value" "2k2/62,5mW" (at 97.79 130.81 0)
       (effects (font (size 1.27 1.27)) (justify left))
     )
@@
       (effects (font (size 1.27 1.27)))
     )
-    (property "Value" "49,9R/62,5mW/0402" (at 252.73 157.48 90)
+    (property "Value" "49,9R/62,5mW" (at 252.73 157.48 90)
       (effects (font (size 1.27 1.27)))
     )
@@
       (effects (font (size 1.27 1.27)))
     )
-    (property "Value" "49,9R/62,5mW/0402" (at 252.73 146.05 90)
+    (property "Value" "49,9R/62,5mW" (at 252.73 146.05 90)
       (effects (font (size 1.27 1.27)))
     )
@@
       (effects (font (size 1.27 1.27)) (justify left))
     )
-    (property "Value" "0,1uF/50V/0402" (at 186.69 43.18 0)
+    (property "Value" "0,1uF/50V" (at 186.69 43.18 0)
       (effects (font (size 1.27 1.27)) (justify left))
     )
@@
       (effects (font (size 1.27 1.27)) (justify left))
     )
-    (property "Value" "12,1k/62,5mW/0402" (at 201.93 118.1099 0)
+    (property "Value" "12,1k/62,5mW" (at 201.93 118.1099 0)
       (effects (font (size 1.27 1.27)) (justify left))
     )
@@
       (effects (font (size 1.27 1.27)) (justify left))
     )
-    (property "Value" "2k2/62,5mW/0402" (at 113.03 53.34 0)
+    (property "Value" "2k2/62,5mW" (at 113.03 53.34 0)
       (effects (font (size 1.27 1.27)) (justify left))
     )
@@
       (effects (font (size 1.27 1.27)) (justify left))
     )
-    (property "Value" "2k2/62,5mW/0402" (at 40.64 53.34 0)
-      (effects (font (size 1.27 1.27)) (justify left))
-    )
+    (property "Value" "2k2/62,5mW" (at 40.64 53.34 0)
+      (effects (font (size 1.27 1.27)) (justify left))
+    )

Commit message: Development
Parts:
- removed J7: ETHERNET, Tales:RJ45_HanRun_HR911105A, symbol Tales:HanRun_HR911105A
- added J1: RJ45 JACK, Tales:RJ45_UDE_RB1-ZZ-0206, symbol Tales:RJ45_UDE_RB1-ZZ-0206
Connections:
- net +3.3VA: now also J1.4 (CT), J1.5 (CT), J1.L2 (RLED+); no longer R16.1
- net GND: now also R17.2, J1.7
- net LED_G_K: now also R16.2
- net LED_Y_A: now also J1.L4 (LLED+); no longer R17.1
- net RD+: now also J1.3 (RD+)
- net RD-: now also J1.6 (RD-)
- net TD+: now also J1.1 (TD+)
- net TD-: now also J1.2 (TD-)
- net at C14.1: now also J1.15 (SHIELD)
- new net: J1.L3 (LLED-), R17.1
- new net: J1.L1 (RLED-), R16.1
- new net PoE+: J1.9 (V+)
- new net PoE-: J1.10 (V-)
Other:
- note added: "UDE CORP RB1-ZZ-0266 JLC C409617 1,24 ABRACON MOUSER 815-ARJP11AMAFMU2 9,05 CUI DEVICES MOUSER 490-CRJ005-M1-TH 5,67 NÃO TEM DIODOS INTERNOS"
- moved on the sheet: C14, C15, C16, C18, C20, C21, C22, R15, R16, R17, R18, R19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
