File: V1/esp-poe-2rl-V1-mcu.kicad_sch (KiCad schematic)
At the start: 10 parts, among them Q3 UMH3N, SW1 RESET, U3 CH340C, U4 ESP32-WROOM-32UE-N16

Commit message: Dev
Other:
- title: ESP 16x 24VDC Input 16x 24VDC Output Module -> ESP 2x Relay Output Module with PoE
Changed lines of the file:
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@@
   (paper "A4")
   (title_block
-    (title "ESP 16x 24VDC Input 16x 24VDC Output Module")
-    (date "2023-05-05")
-    (rev "V2")
+    (title "ESP 2x Relay Output Module with PoE")
+    (date "2023-08-02")
+    (rev "V1")
   )
   (junction (at 63.5 53.34) (diameter 0) (color 0 0 0 0)

Commit message: Working on PoE frontend.
Parts:
- C11: value 10uF/10V/0603 -> 10uF/10V
- C12: value 0,1uF/50V/0805 -> 0,1uF/50V
- C13: value 1uF/50V/0603 -> 1uF/50V
- R10, R11, R12: value 10k/62,5mW/0402 -> 10k/62,5mW
Changed lines of the file:
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@@
       (effects (font (size 1.27 1.27)) (justify left))
     )
-    (property "Value" "1uF/50V/0603" (at 135.89 86.3662 0)
+    (property "Value" "1uF/50V" (at 135.89 86.3662 0)
       (effects (font (size 1.27 1.27)) (justify left))
     )
@@
       (effects (font (size 1.27 1.27)) (justify right))
     )
-    (property "Value" "10k/62,5mW/0402" (at 207.01 69.85 0)
+    (property "Value" "10k/62,5mW" (at 207.01 69.85 0)
       (effects (font (size 1.27 1.27)) (justify right))
     )
@@
       (effects (font (size 1.27 1.27)) (justify left))
     )
-    (property "Value" "10k/62,5mW/0402" (at 227.33 104.14 0)
+    (property "Value" "10k/62,5mW" (at 227.33 104.14 0)
       (effects (font (size 1.27 1.27)) (justify left))
     )
@@
       (effects (font (size 1.27 1.27)) (justify left))
     )
-    (property "Value" "10uF/10V/0603" (at 24.13 60.96 0)
+    (property "Value" "10uF/10V" (at 24.13 60.96 0)
       (effects (font (size 1.27 1.27)) (justify left))
     )
@@
       (effects (font (size 1.27 1.27)) (justify left))
     )
-    (property "Value" "10k/62,5mW/0402" (at 135.89 69.85 0)
+    (property "Value" "10k/62,5mW" (at 135.89 69.85 0)
       (effects (font (size 1.27 1.27)) (justify left))
     )
@@
       (effects (font (size 1.27 1.27)) (justify left))
     )
-    (property "Value" "0,1uF/50V/0805" (at 45.72 60.96 0)
-      (effects (font (size 1.27 1.27)) (justify left))
-    )
+    (property "Value" "0,1uF/50V" (at 45.72 60.96 0)
+      (effects (font (size 1.27 1.27)) (justify left))
+    )

Commit message: Development
Parts:
- added D39, D40: GREEN, Tales:LED_0603_1608Metric, symbol Device:LED_Small
- added Q4, Q5: MMBT2222A, Tales:SOT-23, symbol Device:Q_NPN_BEC
- added R81, R82: 10k/62,5mW, Tales:R_0402_1005Metric, symbol Device:R_US
- added R85, R86: 1k/62,5mW, Tales:R_0402_1005Metric, symbol Device:R_US
- added R89, R90: 5,6k/0,1W, Tales:R_0603_1608Metric, symbol Device:R_US
Connections:
- net GND: now also Q4.2 (E), Q5.2 (E), R81.2, R82.2
- new net: D39.2 (A), R89.2
- new net: Q4.1 (B), R85.1
- new net: Q5.1 (B), R86.1
- new net: D40.2 (A), R90.2
- new net +24V: R89.1, R90.1
- new net J8-OUT1: D39.1 (K), Q4.3 (C)
- new net J8-OUT2: D40.1 (K), Q5.3 (C)
- new net OUT1: R81.1, R85.2
- new net OUT2: R82.1, R86.2
Other:
- moved on the sheet: C11, C12, C13, Q3A, Q3B, R10, R11, R12, SW1, U4

Commit message: Development continues!
Parts:
- renumbered D39 to D1, D40 to D8, R81 to R35, R82 to R36, R85 to R37, R86 to R38, R89 to R39, R90 to R40
Connections:
- net OUT1 is gone; now on an unnamed net: R35.1, R37.2
- net OUT2 is gone; now on an unnamed net: R36.1, R38.2
- no-connect marks 24 -> 22
Changed lines of the file:
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@@
   (no_connect (at 144.78 85.09))
   (no_connect (at 53.34 78.74))
-  (no_connect (at 175.26 133.35))
   (no_connect (at 144.78 115.57))
   (no_connect (at 144.78 118.11))
   (no_connect (at 73.66 88.9))
   (no_connect (at 175.26 97.79))
-  (no_connect (at 175.26 130.81))
   (no_connect (at 175.26 135.89))
   (no_connect (at 73.66 83.82))
@@
     (stroke (width 0) (type default))
   )
+  (wire (pts (xy 219.71 133.35) (xy 219.71 147.32))
+    (stroke (width 0) (type default))
+  )
   (wire (pts (xy 233.68 110.49) (xy 241.3 110.49))
     (stroke (width 0) (type default))
@@
     (stroke (width 0) (type default))
   )
+  (wire (pts (xy 219.71 130.81) (xy 219.71 110.49))
+    (stroke (width 0) (type default))
+  )
   (wire (pts (xy 78.74 49.53) (xy 78.74 78.74))
     (stroke (width 0) (type default))
@@
     (stroke (width 0) (type default))
   )
+  (wire (pts (xy 175.26 130.81) (xy 219.71 130.81))
+    (stroke (width 0) (type default))
+  )
   (wire (pts (xy 264.16 104.14) (xy 257.81 104.14))
     (stroke (width 0) (type default))
@@
     (stroke (width 0) (type default))
   )
-  (wire (pts (xy 231.14 147.32) (xy 233.68 147.32))
-    (stroke (width 0) (type default))
-  )
   (wire (pts (xy 29.21 53.34) (xy 48.26 53.34))
     (stroke (width 0) (type default))
@@
     (stroke (width 0) (type default))
   )
+  (wire (pts (xy 175.26 133.35) (xy 219.71 133.35))
+    (stroke (width 0) (type default))
+  )
   (wire (pts (xy 175.26 113.03) (xy 177.8 113.03))
     (stroke (width 0) (type default))
@@
     (stroke (width 0) (type default))
   )
-  (wire (pts (xy 231.14 110.49) (xy 233.68 110.49))
+  (wire (pts (xy 219.71 110.49) (xy 233.68 110.49))
     (stroke (width 0) (type default))
   )
@@
   )
   (wire (pts (xy 114.3 80.01) (xy 121.92 80.01))
+    (stroke (width 0) (type default))
+  )
+  (wire (pts (xy 219.71 147.32) (xy 233.68 147.32))
     (stroke (width 0) (type default))
   )
@@
     (effects (font (size 1.27 1.27)) (justify left))
   )
-  (hierarchical_label "OUT1" (shape input) (at 231.14 110.49 180) (fields_autoplaced)
-    (effects (font (size 1.27 1.27)) (justify right))
-  )
   (hierarchical_label "J8-OUT2" (shape input) (at 264.16 140.97 0) (fields_autoplaced)
     (effects (font (size 1.27 1.27)) (justify left))
@@
     (effects (font (size 1.27 1.27)) (justify left))
   )
-  (hierarchical_label "OUT2" (shape input) (at 231.14 147.32 180) (fields_autoplaced)
-    (effects (font (size 1.27 1.27)) (justify right))
-  )
   (hierarchical_label "USB_D+" (shape input) (at 38.1 83.82 180) (fields_autoplaced)
     (effects (font (size 1.27 1.27)) (justify right))
@@
   (symbol (lib_id "Device:LED_Small") (at 257.81 100.33 90) (unit 1)
     (in_bom yes) (on_board yes) (dnp no)
-    (property "Reference" "D39" (at 255.27 97.79 90)
+    (property "Reference" "D1" (at 255.27 97.79 90)
       (effects (font (size 1.27 1.27)) (justify left))
     )
@@
   (symbol (lib_id "power:GND") (at 257.81 115.57 0) (unit 1)
     (in_bom yes) (on_board yes) (dnp no)
-    (property "Reference" "#PWR0142" (at 257.81 121.92 0)
+    (property "Reference" "#PWR065" (at 257.81 121.92 0)
       (effects (font (size 1.27 1.27)) hide)
     )
@@
   (symbol (lib_id "power:+24V") (at 257.81 88.9 0) (unit 1)
     (in_bom yes) (on_board yes) (dnp no)
-    (property "Reference" "#PWR0141" (at 257.81 92.71 0)
+    (property "Reference" "#PWR064" (at 257.81 92.71 0)
       (effects (font (size 1.27 1.27)) hide)
     )
@@
   (symbol (lib_id "power:GND") (at 233.68 120.65 0) (unit 1)
     (in_bom yes) (on_board yes) (dnp no)
-    (property "Reference" "#PWR0137" (at 233.68 127 0)
+    (property "Reference" "#PWR034" (at 233.68 127 0)
       (effects (font (size 1.27 1.27)) hide)
     )
@@
   (symbol (lib_id "Device:R_US") (at 257.81 92.71 0) (unit 1)
     (in_bom yes) (on_board yes) (dnp no)
-    (property "Reference" "R89" (at 260.35 90.17 0)
+    (property "Reference" "R39" (at 260.35 90.17 0)
       (effects (font (size 1.27 1.27)) (justify left))
     )
@@
   (symbol (lib_id "Device:R_US") (at 233.68 115.57 0) (unit 1)
     (in_bom yes) (on_board yes) (dnp no)
-    (property "Reference" "R81" (at 236.22 116.84 0)
+    (property "Reference" "R35" (at 236.22 116.84 0)
       (effects (font (size 1.27 1.27)) (justify left))
     )
@@
   (symbol (lib_id "power:+24V") (at 257.81 125.73 0) (unit 1)
     (in_bom yes) (on_board yes) (dnp no)
-    (property "Reference" "#PWR0143" (at 257.81 129.54 0)
+    (property "Reference" "#PWR066" (at 257.81 129.54 0)
       (effects (font (size 1.27 1.27)) hide)
     )
@@
   (symbol (lib_id "Device:R_US") (at 257.81 129.54 0) (unit 1)
     (in_bom yes) (on_board yes) (dnp no)
-    (property "Reference" "R90" (at 260.35 127 0)
+    (property "Reference" "R40" (at 260.35 127 0)
       (effects (font (size 1.27 1.27)) (justify left))
     )
@@
   (symbol (lib_id "Device:R_US") (at 245.11 110.49 270) (unit 1)
     (in_bom yes) (on_board yes) (dnp no)
-    (property "Reference" "R85" (at 245.11 105.41 90)
+    (property "Reference" "R37" (at 245.11 105.41 90)
       (effects (font (size 1.27 1.27)))
     )
@@
   (symbol (lib_id "power:GND") (at 233.68 157.48 0) (unit 1)
     (in_bom yes) (on_board yes) (dnp no)
-    (property "Reference" "#PWR0138" (at 233.68 163.83 0)
+    (property "Reference" "#PWR035" (at 233.68 163.83 0)
       (effects (font (size 1.27 1.27)) hide)
     )
@@
   (symbol (lib_id "Device:LED_Small") (at 257.81 137.16 90) (unit 1)
     (in_bom yes) (on_board yes) (dnp no)
-    (property "Reference" "D40" (at 255.27 134.62 90)
+    (property "Reference" "D8" (at 255.27 134.62 90)
       (effects (font (size 1.27 1.27)) (justify left))
     )
@@
   (symbol (lib_id "power:GND") (at 257.81 152.4 0) (unit 1)
     (in_bom yes) (on_board yes) (dnp no)
-    (property "Reference" "#PWR0144" (at 257.81 158.75 0)
+    (property "Reference" "#PWR067" (at 257.81 158.75 0)
       (effects (font (size 1.27 1.27)) hide)
     )
@@
   (symbol (lib_id "Device:R_US") (at 233.68 152.4 0) (unit 1)
     (in_bom yes) (on_board yes) (dnp no)
-    (property "Reference" "R82" (at 236.22 153.67 0)
+    (property "Reference" "R36" (at 236.22 153.67 0)
       (effects (font (size 1.27 1.27)) (justify left))
     )
@@
   (symbol (lib_id "Device:R_US") (at 245.11 147.32 270) (unit 1)
     (in_bom yes) (on_board yes) (dnp no)
-    (property "Reference" "R86" (at 245.11 142.24 90)
+    (property "Reference" "R38" (at 245.11 142.24 90)
       (effects (font (size 1.27 1.27)))
     )
