File: V1/esp-poe-2rl-V1-backup.kicad_pcb (KiCad board)
At the start: 2 copper layers, 89 x 45 mm, 88 parts, among them J1 USB_C_Receptacle_USB2.0, J2 RJ45 JACK, J3 1x2P 5,08mm, J4 1x2P 5,08mm, K1 G5NB-1A-E-DC5, K2 G5NB-1A-E-DC5, Q1 UMH3N, Q2 WPM2015-3/TR, Q3 LMUN2211LT1G, Q4 MMBT2222A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

Commit message: Last touches
Parts:
- moved C1 4.00 mm to (147.0, 110.0)
- moved C2 4.00 mm to (163.5, 108.3)
- moved C3 4.00 mm to (153.5, 96.0)
- moved C4 4.00 mm to (149.2, 99.5)
- moved C5 4.00 mm to (147.0, 82.3)
- moved C6 4.00 mm to (167.0, 75.2)
- moved C7 4.00 mm to (156.0, 75.5)
- moved C8 4.00 mm to (144.0, 75.0)
- moved C9 4.00 mm to (150.0, 75.0)
- moved D1 4.00 mm to (144.0, 109.0)
- moved D2 4.00 mm to (152.5, 90.5)
- moved D3 4.00 mm to (164.5, 83.0)
- moved D4 4.00 mm to (160.0, 83.0)
- moved D5 4.00 mm to (154.7, 80.5)
- moved F1 4.00 mm to (154.6, 85.0)
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Routing:
- net PoE-: track 37.9 -> 19.6 mm, vias 3 -> 0
- net +3.3V: track 117.0 -> 103.0 mm, vias 6 -> 5
- net Net-(C10-Pad1): track 73.2 -> 62.8 mm
- net +5V: track 128.6 -> 135.3 mm
- net PoE+: track 65.6 -> 62.3 mm, vias 3 -> 0
- net OUT1: track 20.0 -> 22.0 mm
- net GND: track 113.2 -> 115.2 mm
- net +3.3VLAN: track 46.6 -> 48.1 mm
- net /EMAC_RXD1: track 40.2 -> 41.1 mm
- net /EMAC_RXD0: track 38.3 -> 39.1 mm
- net PG: track 38.0 -> 38.7 mm
- net Net-(Q1A-C1): track 31.3 -> 31.9 mm
- net /TD+: track 21.4 -> 21.9 mm
Other:
- board size 89 x 45 mm -> 93 x 45 mm
