File: V1/eumesmo-poe-2rl-v1.kicad_pcb (KiCad board)
At the start: 4 copper layers, 82.5 x 45 mm, 109 parts, among them J1 USB_C_Receptacle_USB2.0, J2 RJ45 JACK, J3 250-202, J4 250-202, K1 G5NB-1A-E-DC5, K2 G5NB-1A-E-DC5, Q1 UMH3N, Q2 WPM2015-3/TR, Q3 LMUN2211LT1G, Q4 MMBT2222A, Q5 MMBT2222A, SW1 RESET, U1 CH340K, U2 ESP32-WROOM-32UE-N16, U3 LAN8710A, U4 TPS2376DDAR-H, U5 TX4138, U6 SY8089A1AAC

Commit message: Added CPU health LED
Other:
- board text added: "V1.6 2026-07-02"
- board text removed: "V1.5 2026-06-17"
Changed lines of the file:
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@@
 		)
 	)
-	(gr_text "V1.5 2026-06-17"
+	(gr_text "V1.6 2026-07-02"
 		(at 141 114.375 0)
 		(layer "F.SilkS")
